Commit message: change something

File: ur5/urdfs/ur5_robotiq_140.urdf (robot description, URDF)
Before this commit: robot ur5_robotiq_140, 20 links, 19 joints
Joints:
- removed joint finger_joint
- added joint left_outer_knuckle_joint: type revolute, parent robotiq_arg2f_base_link, child left_outer_knuckle, origin xyz=0 -0.030601 0.054905 rpy=2.2957963267948966 0 0, axis -1 0 0, limit lower=0 upper=0.7 effort=1000 velocity=2.0
- joint left_inner_finger_joint: mimic joint=finger_joint multiplier=1 offset=0 -> joint=left_outer_knuckle_joint multiplier=1 offset=0
- joint left_inner_knuckle_joint: mimic joint=finger_joint multiplier=-1 offset=0 -> joint=left_outer_knuckle_joint multiplier=-1 offset=0
- joint right_inner_finger_joint: mimic joint=finger_joint multiplier=1 offset=0 -> joint=left_outer_knuckle_joint multiplier=1 offset=0
- joint right_inner_knuckle_joint: mimic joint=finger_joint multiplier=-1 offset=0 -> joint=left_outer_knuckle_joint multiplier=-1 offset=0
- joint right_outer_knuckle_joint: mimic joint=finger_joint multiplier=-1 offset=0 -> joint=left_outer_knuckle_joint multiplier=-1 offset=0
